Commit message: small changes

File: urdf/lcube_car.urdf (robot description, URDF)
Before this commit: robot lcube, 28 links, 27 joints
Links:
- removed link back_camera_link
- removed link back_camera_link_optical
- removed link back_left_far_sonar_link
- removed link back_left_middle_sonar_link
- removed link back_right_far_sonar_link
- removed link back_right_middle_sonar_link
- removed link base_link
- removed link center_laser_link
- removed link front_camera_link
- removed link front_camera_link_optical
- removed link front_left_far_sonar_link
- removed link front_left_laser_link
- removed link front_left_middle_sonar_link
- removed link front_right_far_sonar_link
- removed link front_right_laser_link
- removed link front_right_middle_sonar_link
- removed link left_camera_link
- removed link left_camera_link_optical
- removed link right_camera_link
- removed link right_camera_link_optical
- link chassis: geometry collision box size=1.168381 1.654253 0.272347; collision box size=1.267845 1.116344 0.244286
- link front_left_wheel: geometry collision sphere radius=0.31265; visual mesh filename=package://lcube_test_description/meshes/wheel.obj scale=0.01 0.01 0.01
- link front_right_wheel: geometry collision sphere radius=0.31265; visual mesh filename=package://lcube_test_description/meshes/wheel.obj scale=0.01 0.01 0.01
- link rear_left_wheel: geometry collision sphere radius=0.31265; visual mesh filename=package://lcube_test_description/meshes/wheel.obj scale=0.01 0.01 0.01
- link rear_right_wheel: geometry collision sphere radius=0.31265; visual mesh filename=package://lcube_test_description/meshes/wheel.obj scale=0.01 0.01 0.01
- link steering_wheel: geometry visual mesh filename=package://lcube_test_description/meshes/steering_wheel.obj scale=0.01 0.01 0.01
Joints:
- removed joint back_camera_joint
- removed joint back_camera_optical_joint
- removed joint back_left_far_sonar_joint
- removed joint back_left_middle_sonar_joint
- removed joint back_right_far_sonar_joint
- removed joint back_right_middle_sonar_joint
- removed joint base_link_connection
- removed joint center_laser_joint
- removed joint front_camera_joint
- removed joint front_camera_optical_joint
- removed joint front_left_far_sonar_joint
- removed joint front_left_laser_joint
- removed joint front_left_middle_sonar_joint
- removed joint front_right_far_sonar_joint
- removed joint front_right_laser_joint
- removed joint front_right_middle_sonar_joint
- removed joint left_camera_joint
- removed joint left_camera_optical_joint
- removed joint right_camera_joint
- removed joint right_camera_optical_joint

Commit message: new world

File: urdf/lcube_car.urdf (robot description, URDF)
Before this commit: robot lcube, 8 links, 7 joints
Links:
- link chassis: geometry collision box size=1.168381 1.654253 0.272347; collision box size=1.267845 1.116344 0.244286
- link front_left_wheel: geometry collision sphere radius=0.31265; visual mesh filename=package://prius/meshes/wheel.obj scale=0.01 0.01 0.01
- link front_right_wheel: geometry collision sphere radius=0.31265; visual mesh filename=package://prius/meshes/wheel.obj scale=0.01 0.01 0.01
- link rear_left_wheel: geometry collision sphere radius=0.31265; visual mesh filename=package://prius/meshes/wheel.obj scale=0.01 0.01 0.01
- link rear_right_wheel: geometry collision sphere radius=0.31265; visual mesh filename=package://prius/meshes/wheel.obj scale=0.01 0.01 0.01
- link steering_wheel: geometry visual mesh filename=package://prius/meshes/steering_wheel.obj scale=0.01 0.01 0.01
